File: Ksawer_Krzysztof.kicad_sch (KiCad schematic)
At the start: 35 parts, among them K1 1461103-1, K2 1461103-1, Q1 BC547, Q2 MMBT3904, Q3 MMBT3904, U1 DHT11, U2 ESP-12E, U3 NHD-C0220BIZ, U4 LTV-844, U5 STM32F038K6Ux

Commit message: ślady stoopek
Dwa slady w przekaźnikach, są jakieś ostrzeżenia
Parts:
- K1, K2: footprint (none) -> Trans_footprint:OJ_OJE_Relay
- U4: footprint Package_DIP:DIP-16_W7.62mm -> Trans_footprint:SSO-16_P2.54
Changed lines of the file:
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@@
       (effects (font (size 1.27 1.27)) (justify left))
     )
-    (property "Footprint" "" (at 186.69 149.86 0)
+    (property "Footprint" "Trans_footprint:OJ_OJE_Relay" (at 186.69 149.86 0)
       (effects (font (size 1.27 1.27)) (justify left) hide)
     )
@@
       (effects (font (size 1.27 1.27)) (justify left))
     )
-    (property "Footprint" "" (at 93.98 154.94 0)
-      (effects (font (size 1.27 1.27)) (justify left) hide)
+    (property "Footprint" "Trans_footprint:OJ_OJE_Relay" (at 93.98 154.94 0)
+      (effects (font (size 1.27 1.27)) (justify left))
     )
     (property "Datasheet" "" (at 100.33 157.48 0)
@@
       (effects (font (size 1.27 1.27)))
     )
-    (property "Footprint" "Package_DIP:DIP-16_W7.62mm" (at 27.94 172.72 0)
+    (property "Footprint" "Trans_footprint:SSO-16_P2.54" (at 27.94 172.72 0)
       (effects (font (size 1.27 1.27) italic) (justify left) hide)
     )
@@
       (effects (font (size 1.27 1.27)))
     )
-    (property "Footprint" "Package_DIP:DIP-16_W7.62mm" (at 120.65 167.64 0)
+    (property "Footprint" "Trans_footprint:SSO-16_P2.54" (at 120.65 167.64 0)
       (effects (font (size 1.27 1.27) italic) (justify left) hide)
     )

Commit message: zmiany2
Parts:
- added C10: 1uf, symbol Device:C
- added C11, C12: 18pf, symbol Device:C
- added C7: 4,7uf, symbol Device:C
- added C8: 100nf, symbol Device:C
- added C9: 10nf, symbol Device:C
- added Y1: ABM3-B.000MHZ-D2Y, symbol Device:Crystal
Connections:
- net GND: now also C6.2, U5.31 (BOOT0), C10.2, C11.2, C12.2, C7.2, C8.2, C9.2
- net VDD: now also U5.1 (VDD), U5.5 (VDDA), C10.1, C7.1, C8.1, C9.1; no longer U5.17 (VDD)
- net at U5.2 (PF0): now also C11.1, Y1.2
- net at U5.3 (PF1): now also C12.1, Y1.1
- no-connect marks 13 -> 30
Other:
- note added: "MCU"
- moved on the sheet: C6, U5

Commit message: zmiana3
Parts:
- added C13: 0.1uf, symbol Device:C
Connections:
- net VCC is gone; now on net VDD: BZ1.1 (-), D1.1 (K), R3.1, R5.1, U1.1 (VDD)
- net GND: now also C13.1
- net VDD: no longer C10.1, C9.1, U5.5 (VDDA)
- net at U5.16 (NPOR): now also C13.2
- net RST: no longer names the net of U3.1 (~{RST})
- new net VDDA: C10.1, C9.1, U5.5 (VDDA)
Other:
- moved on the sheet: C10, C11, C12, C6, C7, C8, C9, D2, D3, K1, K2, Q2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

Commit message: koniec bez błedów
koniec bez błedów
Parts:
- added C14, C15, C16: 10 uF 1mR, symbol Device:C
- added C17: 22uF 1mR, symbol Device:C
- added C18: 100nF 1mR, symbol Device:C
- added D4: BAT54S, Package_TO_SOT_SMD:SOT-23, symbol Diode:BAT54S
- added J1: BAT, symbol Connector_Generic:Conn_01x02
- added J3: V1, symbol Connector_Generic:Conn_01x03
- added L1: 1uH 57mR, symbol Device:L
- added R16, R17: 100K, symbol Device:R
- added R18: 200R, symbol Device:R
- added U6: TPS63021DSJR, TPS63021DSJR:IC_TPS63021DSJR, symbol TPS63021DSJR:TPS63021DSJR
- added U8: INA180A1, Package_TO_SOT_SMD:SOT-23-5, symbol Amplifier_Current:INA180A1
Connections:
- net COM_V1: now also J3.2 (Pin_2)
- net GND: now also C14.2, C15.2, C16.2, C17.2, C18.2, D4.1 (A), J1.1 (Pin_1), R17.2, U6.13 (PS/SYNC), U6.15 (PGND), U6.2 (GND), U8.2 (GND)
- net Relay1_NO: now also J3.1 (Pin_1)
- net Relay2_NO: now also J3.3 (Pin_3)
- net VDD: now also C14.1, C15.1, C16.1, D4.2 (K), U6.3 (FB), U6.4 (VOUT_4), U6.5 (VOUT_5), U8.5 (V+)
- net VBAT_ADC: now reaches U5.6 (PA0)
- net VBAT_ADC: now also R18.1
- new net: D4.3 (COM), R18.2, U8.1, U8.4 (-)
- new net: C18.1, U6.1 (VINA), U6.12 (EN)
- new net: L1.2, U6.6 (L2_6), U6.7 (L2_7)
- new net: L1.1, U6.8 (L1_8), U6.9 (L1_9)
- new net: R16.2, R17.1, U8.3 (+)
- new net +BATT: C17.1, J1.2 (Pin_2), R16.1, U6.10 (VIN_10), U6.11 (VIN_11)
Other:
- note added: "PSU"
- moved on the sheet: D3, K2, Q3, R13, R15, U4B

Commit message: zmiana4
Parts:
- BZ1: footprint (none) -> Buzzer_Beeper:Buzzer_12x9.5RM7.6
- C1, C10, C11, C12, C13, C14, C15, C16, C17, C18, C2, C3, C4, C5, C6, C7, C8, C9: footprint (none) -> Capacitor_SMD:C_0603_1608Metric_Pad1.08x0.95mm_HandSolder
- J1: footprint (none) -> Connector_PinHeader_1.00mm:PinHeader_1x02_P1.00mm_Vertical
- J3: footprint (none) -> Connector_PinHeader_1.00mm:PinHeader_1x03_P1.00mm_Vertical
- L1: footprint (none) -> Inductor_SMD:L_0603_1608Metric
- R1, R10, R11, R12, R13, R14, R15, R16, R17, R18, R2, R3, R4, R5, R7, R8, R9: footprint (none) -> Resistor_SMD:R_0805_2012Metric
- Y1: footprint (none) -> Crystal:Crystal_SMD_5032-2Pin_5.0x3.2mm
Other:
- moved on the sheet: J1, J3

Commit message: zmiany
Parts:
- U6: footprint TPS63021DSJR:IC_TPS63021DSJR -> IC:IC_TPS63021DSJR
Changed lines of the file:
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@@
       (effects (font (size 1.27 1.27)))
     )
-    (property "Footprint" "TPS63021DSJR:IC_TPS63021DSJR" (at 228.6 123.19 0)
+    (property "Footprint" "IC:IC_TPS63021DSJR" (at 228.6 123.19 0)
       (effects (font (size 1.27 1.27)) (justify bottom) hide)
     )

Commit message: lab3
lab3
Parts:
- R6: value LDR23 -> LDR1; footprint 500mW; 50÷100kΩ; 560nm; THT; ØLED: 20mm; -> Trans_footprint:LDR
Connections:
- net COM_V1: now also U4.10; no longer U4.14
- net GND: now also U4.8; no longer U4.4
- net at R15.1: now also U4.9; no longer U4.13
- net at R13.2: now also U4.7; no longer U4.3
Changed lines of the file:
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@@
       (effects (font (size 1.27 1.27)) (justify left))
     )
-    (property "Value" "LDR23" (at 77.47 110.49 0)
-      (effects (font (size 1.27 1.27)) (justify left))
-    )
-    (property "Footprint" "500mW; 50÷100kΩ; 560nm; THT; ØLED: 20mm;" (at 79.375 109.22 90)
-      (effects (font (size 1.27 1.27)) hide)
-    )
-    (property "Datasheet" "https://www.tme.eu/pl/details/02-ldr23/fotorezystory/nte-electronics/?brutto=1&currency=PLN&gad_source=1&gclid=CjwKCAiAgeeqBhBAEiwAoDDhnxxvvgZ09eV3et7v3hX89EgXv7xleamlIjj7GZW6hUo37maD1W62bxoCXXIQAvD_BwE" (at 74.93 110.49 0)
+    (property "Value" "LDR1" (at 77.47 110.49 0)
+      (effects (font (size 1.27 1.27)) (justify left))
+    )
+    (property "Footprint" "Trans_footprint:LDR" (at 79.375 109.22 90)
+      (effects (font (size 1.27 1.27)) hide)
+    )
+    (property "Datasheet" "https://www.tme.eu/pl/details/02-ldr21/fotorezystory/nte-electronics/" (at 74.93 110.49 0)
       (effects (font (size 1.27 1.27)) hide)
     )
@@
     )
   )
-  (symbol (lib_id "Isolator:LTV-844") (at 77.47 180.34 0) (unit 2)
+  (symbol (lib_id "Isolator:LTV-844") (at 77.47 180.34 0) (unit 4)
     (in_bom yes) (on_board yes) (dnp no) (fields_autoplaced)
     (property "Reference" "U4" (at 77.47 171.45 0)
@@
       (project "Ksawer_Krzysztof"
         (path "/1467245e-82c5-4f8a-9413-861f78518855"
-          (reference "U4") (unit 2)
-        )
-      )
+          (reference "U4") (unit 4)
+        )
+      )

Commit message: polaczenia ale nie wiem czy to wg ma sens
Connections:
- net +BATT: now also C18.1, U6.12 (EN)
- now unconnected: U6.1 (VINA)
- no-connect marks 30 -> 32
Changed lines of the file:
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@@
   (junction (at 199.39 123.19) (diameter 0) (color 0 0 0 0)
   )
+  (junction (at 199.39 115.57) (diameter 0) (color 0 0 0 0)
+  )
   (junction (at 247.65 140.97) (diameter 0) (color 0 0 0 0)
   )
@@
   (junction (at 48.26 71.12) (diameter 0) (color 0 0 0 0)
   )
-  (junction (at 209.55 115.57) (diameter 0) (color 0 0 0 0)
-  )
   (junction (at 124.46 92.71) (diameter 0) (color 0 0 0 0)
   )
@@
   (no_connect (at 256.54 72.39))
   (no_connect (at 256.54 67.31))
+  (no_connect (at 210.82 115.57))
   (no_connect (at 33.02 62.23))
   (no_connect (at 228.6 74.93))
@@
   (no_connect (at 246.38 120.65))
   (no_connect (at 228.6 72.39))
+  (no_connect (at 219.71 134.62))
   (no_connect (at 243.84 36.83))
   (wire (pts (xy 252.73 30.48) (xy 260.35 30.48))
@@
     (stroke (width 0) (type default))
   )
-  (wire (pts (xy 210.82 120.65) (xy 209.55 120.65))
+  (wire (pts (xy 210.82 120.65) (xy 208.28 120.65))
     (stroke (width 0) (type default))
   )
@@
     (stroke (width 0) (type default))
   )
-  (wire (pts (xy 209.55 120.65) (xy 209.55 115.57))
+  (wire (pts (xy 208.28 120.65) (xy 208.28 115.57))
     (stroke (width 0) (type default))
   )
@@
     (stroke (width 0) (type default))
   )
-  (wire (pts (xy 210.82 115.57) (xy 209.55 115.57))
-    (stroke (width 0) (type default))
-  )
   (polyline (pts (xy 181.61 123.19) (xy 181.61 124.46))
     (stroke (width 0) (type dash))
@@
     (stroke (width 0) (type default))
   )
-  (wire (pts (xy 209.55 115.57) (xy 199.39 115.57))
+  (wire (pts (xy 208.28 115.57) (xy 199.39 115.57))
     (stroke (width 0) (type default))
   )
@@
     (stroke (width 0) (type default))
   )
+  (wire (pts (xy 195.58 115.57) (xy 199.39 115.57))
+    (stroke (width 0) (type default))
+  )
   (polyline (pts (xy 181.61 123.19) (xy 181.61 124.46))
     (stroke (width 0) (type dash))
@@
         )
       )
+    )
+  )
+  (symbol (lib_id "power:+BATT") (at 195.58 115.57 0) (unit 1)
+    (in_bom yes) (on_board yes) (dnp no)
+    (property "Reference" "#PWR038" (at 195.58 119.38 0)
+      (effects (font (size 1.27 1.27)) hide)
+    )
+    (property "Value" "+BATT" (at 194.31 111.76 0)
+      (effects (font (size 1.27 1.27)))
+    )
+    (property "Footprint" "" (at 195.58 115.57 0)
+      (effects (font (size 1.27 1.27)) hide)
+    )
+    (property "Datasheet" "" (at 195.58 115.57 0)
+      (effects (font (size 1.27 1.27)) hide)
+    )
+    (pin "1")
+    (instances
+      (project "Ksawer_Krzysztof"
+        (path "/1467245e-82c5-4f8a-9413-861f78518855"
+          (reference "#PWR038") (unit 1)
+        )
+      )
