File: Ksawer_Krzysztof.kicad_sch (KiCad schematic)
At the start: 57 parts, among them J1 BAT, J3 V1, K1 1461103-1, K2 1461103-1, Q1 BC547, Q2 MMBT3904, Q3 MMBT3904, U1 DHT11, U2 ESP-12E, U3 NHD-C0220BIZ, U4 LTV-844, U5 STM32F038K6Ux, U6 TPS63021DSJR, U8 INA180A1, Y1 ABM3-B.000MHZ-D2Y

Commit message: prawie koniec
Parts:
- U3: footprint Display:NHD-C0220BiZ -> Trans_footprint:NHD-C0220BiZ
Changed lines of the file:
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@@
       (effects (font (size 1.27 1.27)) (justify left))
     )
-    (property "Footprint" "Display:NHD-C0220BiZ" (at 142.24 62.23 0)
+    (property "Footprint" "Trans_footprint:NHD-C0220BiZ" (at 142.24 62.23 0)
       (effects (font (size 1.27 1.27)) hide)
     )

Commit message: iok
Parts:
- C13: value 0.1uf -> 100nf
Other:
- company: (none) -> Ksawery Giera & Krzysztof Nosal
- title: (none) -> Prototyp układu automatycznej kiełkownicy
Changed lines of the file:
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@@
 (kicad_sch (version 20230121) (generator eeschema)
   (paper "A4")
+  (title_block
+    (title "Prototyp układu automatycznej kiełkownicy")
+    (date "15.12.2023")
+    (rev "v1.1")
+    (company "Ksawery Giera & Krzysztof Nosal")
+  )
   (junction (at 260.35 30.48) (diameter 0) (color 0 0 0 0)
   )
@@
       (effects (font (size 1.27 1.27)) (justify left))
     )
-    (property "Value" "0.1uf" (at 219.71 50.8 90)
+    (property "Value" "100nf" (at 219.71 50.8 90)
       (effects (font (size 1.27 1.27)) (justify left))
     )

Commit message: uj
Parts:
- C14, C15, C16: value 10 uF 1mR -> 10uF
- C17: value 22uF 1mR -> 22uF
- C18: value 100nF 1mR -> 100nF
Changed lines of the file:
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@@
       (effects (font (size 1.27 1.27)) (justify left))
     )
-    (property "Value" "100nF 1mR" (at 200.66 121.92 0)
+    (property "Value" "100nF" (at 200.66 121.92 0)
       (effects (font (size 1.27 1.27)) (justify left))
     )
@@
       (effects (font (size 1.27 1.27)) (justify left))
     )
-    (property "Value" "10 uF 1mR" (at 256.54 119.38 90)
+    (property "Value" "10uF" (at 256.54 114.3 90)
       (effects (font (size 1.27 1.27)) (justify left))
     )
@@
       (effects (font (size 1.27 1.27)) (justify left))
     )
-    (property "Value" "10 uF 1mR" (at 279.4 119.38 90)
+    (property "Value" "10uF" (at 279.4 114.3 90)
       (effects (font (size 1.27 1.27)) (justify left))
     )
@@
   (symbol (lib_id "Device:C") (at 264.16 111.76 0) (unit 1)
     (in_bom yes) (on_board yes) (dnp no)
-    (property "Reference" "C15" (at 260.35 114.3 0)
-      (effects (font (size 1.27 1.27)) (justify left))
-    )
-    (property "Value" "10 uF 1mR" (at 267.97 119.38 90)
+    (property "Reference" "C15" (at 259.08 115.57 0)
+      (effects (font (size 1.27 1.27)) (justify left))
+    )
+    (property "Value" "10uF" (at 267.97 114.3 90)
       (effects (font (size 1.27 1.27)) (justify left))
     )
@@
       (effects (font (size 1.27 1.27)) (justify left))
     )
-    (property "Value" "22uF 1mR" (at 201.93 111.76 0)
-      (effects (font (size 1.27 1.27)) (justify left))
-    )
+    (property "Value" "22uF" (at 203.2 110.49 0)
+      (effects (font (size 1.27 1.27)) (justify left))
+    )
