File: Ksawer_Krzysztof.kicad_pcb (KiCad board)
At the start: 2 copper layers, 57 parts, among them J1 BAT, J3 V1, K1 1461103-1, K2 1461103-1, Q1 BC547, Q2 MMBT3904, Q3 MMBT3904, U1 DHT11, U2 ESP-12E, U3 NHD-C0220BIZ, U4 LTV-844, U5 STM32F038K6Ux, U6 TPS63021DSJR, U8 INA180A1, Y1 ABM3-B.000MHZ-D2Y

Commit message: wstepnie ulozona
Parts:
- moved C16 282.5 mm to (133.1, 118.4), turned to 90 degrees
- moved C15 280.9 mm to (134.9, 118.4), turned to 90 degrees
- moved C14 273.9 mm to (136.7, 118.4), turned to 90 degrees
- moved C13 272.3 mm to (138.3, 105.1), turned to 90 degrees
- moved C17 271.4 mm to (144.0, 118.5), turned to 90 degrees
- moved C12 270.5 mm to (140.1, 105.1), turned to 90 degrees
- moved C8 270.4 mm to (140.1, 101.6), turned to 90 degrees
- moved C18 269.3 mm to (145.9, 118.5), turned to 90 degrees
- moved C9 268.6 mm to (141.9, 101.6), turned to 90 degrees
- moved C11 268.6 mm to (141.9, 105.2), turned to 90 degrees
- moved C7 268.0 mm to (138.3, 101.5), turned to 90 degrees
- moved C10 266.8 mm to (143.7, 101.6), turned to 90 degrees
- moved C5 265.3 mm to (141.3, 91.7), turned to 180 degrees
- moved U2 262.5 mm to (172.1, 109.1)
- moved C6 262.5 mm to (143.7, 105.2), turned to 90 degrees
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
Commit message: pierwsze laczenia
Parts:
- moved J1 54.7 mm to (90.0, 117.4), turned to 180 degrees
- moved C13 38.2 mm to (156.4, 138.7), turned to -90 degrees
- moved C6 38.1 mm to (161.8, 138.7)
- moved C10 38.1 mm to (161.8, 135.2)
- moved C11 38.1 mm to (160.0, 138.7)
- moved C12 38.1 mm to (158.1, 138.7)
- moved C7 38.1 mm to (156.4, 135.1)
- moved C9 38.1 mm to (160.0, 135.2)
- moved C8 38.1 mm to (158.2, 135.1)
- moved C2 11.7 mm to (160.6, 103.3), turned to 180 degrees
- moved R12 11.4 mm to (133.2, 111.3)
- moved Y1 6.90 mm to (142.7, 102.3), turned to 90 degrees
- moved R13 6.82 mm to (133.1, 103.7)
- moved R11 5.75 mm to (148.9, 97.7), turned to -90 degrees
- moved R10 5.54 mm to (151.9, 97.7), turned to -90 degrees
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Routing:
- net /COM_V1: track 0.00 -> 86.0 mm
- net VDD: track 0.00 -> 64.9 mm
- net GND: track 0.00 -> 53.4 mm
- net SCL: track 0.00 -> 16.2 mm
- net SDA: track 0.00 -> 13.1 mm
- net /Relay1_NO: track 0.00 -> 10.0 mm
- net Net-(R15-Pad1): track 0.00 -> 8.64 mm
- net Net-(R12-Pad2): track 0.00 -> 8.43 mm
- net Net-(D2-A): track 0.00 -> 7.66 mm
- net Net-(D3-A): track 0.00 -> 7.62 mm
- net Net-(U2-~{RST}): track 0.00 -> 6.13 mm
- net Net-(U6-L2_6): track 0.00 -> 5.45 mm
- net /Relay2_NO: track 0.00 -> 5.35 mm
- net Net-(U6-L1_8): track 0.00 -> 5.16 mm
- net Net-(R14-Pad1): track 0.00 -> 4.80 mm
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- added copper zone on F.Cu, net +BATT
- added copper zone on F.Cu, net GND
- added copper zone on F.Cu, net VDD

Commit message: polaczenia ale nie wiem czy to wg ma sens
Parts:
- moved C11 48.2 mm to (135.4, 97.3), turned to 180 degrees
- moved C12 45.6 mm to (135.4, 99.2), turned to 180 degrees
- moved C7 41.1 mm to (140.6, 97.1)
- moved C8 41.1 mm to (142.4, 97.1)
- moved C6 37.6 mm to (138.7, 109.0), turned to -90 degrees
- moved C10 33.7 mm to (140.4, 109.0), turned to -90 degrees
- moved C9 31.6 mm to (142.2, 109.0), turned to -90 degrees
- moved C13 30.7 mm to (150.8, 108.5), turned to 90 degrees
- moved R6 13.8 mm to (202.0, 97.5), turned to 180 degrees
- moved R12 12.6 mm to (131.3, 123.8)
- moved R16 10.3 mm to (156.0, 113.6), turned to -90 degrees
- moved D1 9.88 mm to (185.8, 106.8)
- moved BZ1 8.09 mm to (199.9, 115.4), turned to 90 degrees
- moved R18 8.08 mm to (151.1, 116.4), turned to -90 degrees
- moved Q1 7.75 mm to (193.0, 103.5), turned to 90 degrees
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Connections:
- C18 pad 1: Net-(U6-EN) -> +BATT
- U6 pad 1: Net-(U6-EN) -> unconnected-(U6-VINA-Pad1)
- U6 pad 12: Net-(U6-EN) -> +BATT
Routing:
- net Data4: track 0.00 -> 165.1 mm
- net GND: track 53.4 -> 190.8 mm
- net VDD: track 64.9 -> 166.8 mm
- net Data3: track 0.00 -> 95.1 mm
- net Data2: track 0.00 -> 92.3 mm
- net Data1: track 0.00 -> 69.6 mm
- net USART1_RX: track 0.00 -> 61.7 mm
- net USART1_TX: track 0.00 -> 43.2 mm
- net /VBAT_ADC: track 0.00 -> 18.3 mm
- net Net-(U5-NRST): track 0.00 -> 12.0 mm
- net SCL: track 16.2 -> 4.56 mm
- net Net-(D4-COM): track 0.00 -> 10.7 mm
- net Net-(BZ1-+): track 0.00 -> 10.4 mm
- net Net-(U5-PF1): track 4.50 -> 14.1 mm
- net VDDA: track 0.00 -> 9.52 mm
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- added copper zone on F.Cu, net Net-(U6-L1_8)
- added copper zone on F.Cu, net Net-(U6-L2_6)

Commit message: prawie koniec
Parts:
- U3: footprint Display:NHD-C0220BiZ -> Trans_footprint:NHD-C0220BiZ
- moved U3 21.3 mm to (154.0, 93.5)
- moved R6 11.2 mm to (191.3, 100.8)
- moved R12 11.0 mm to (133.5, 113.0)
- moved R10 8.10 mm to (157.2, 101.4), turned to 90 degrees
- moved U1 7.91 mm to (181.6, 93.5)
- moved C5 7.47 mm to (148.0, 95.5)
- moved R11 6.72 mm to (154.4, 100.2), turned to 90 degrees
- moved C4 6.69 mm to (150.4, 96.4)
- moved R16 6.41 mm to (151.2, 117.9), turned to 0 degrees
- moved Q1 4.18 mm to (197.1, 102.6)
- moved R9 4.00 mm to (201.3, 102.3)
- moved R18 1.45 mm to (151.1, 115.0)
Routing:
- net Data4: track 165.1 -> 26.2 mm, vias 0 -> 2
- net GND: track 190.8 -> 57.6 mm, vias 0 -> 23
- net +BATT: track 0.00 -> 64.2 mm, vias 0 -> 2
- net Data2: track 92.3 -> 51.5 mm, vias 0 -> 2
- net VDD: track 166.8 -> 204.5 mm
- net Data3: track 95.1 -> 58.8 mm, vias 0 -> 2
- net Data5: track 0.00 -> 24.2 mm, vias 0 -> 2
- net USART1_RX: track 61.7 -> 40.8 mm, vias 0 -> 2
- net Data1: track 69.6 -> 53.5 mm, vias 0 -> 2
- net SCL: track 4.56 -> 17.1 mm
- net SDA: track 6.69 -> 13.8 mm
- net /VBAT_ADC: track 18.3 -> 13.3 mm
- net Net-(R12-Pad2): track 4.89 -> 7.34 mm
- net Net-(BZ1-+): track 10.4 -> 12.3 mm
- net Net-(D4-COM): track 10.7 -> 11.6 mm
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- added copper zone on B.Cu, net GND
Other:
- board outline added: 119.1 x 37.3 mm

Commit message: warstwa
Parts:
- moved Q1 89.7 mm to (110.0, 81.4)
- moved D1 89.7 mm to (98.6, 85.6)
- moved R6 89.7 mm to (104.1, 79.7)
- moved R9 89.7 mm to (114.1, 81.1)
- moved BZ1 89.7 mm to (112.8, 94.2)
- moved R5 89.7 mm to (99.8, 80.5)
- moved R3 88.7 mm to (96.9, 89.7), turned to 0 degrees
- moved U1 85.3 mm to (96.3, 94.2)
- moved R2 49.2 mm to (120.7, 86.3)
- moved R4 49.0 mm to (143.4, 86.0)
- moved R8 49.0 mm to (143.4, 90.4)
- moved R7 49.0 mm to (143.4, 88.1)
- moved U2 48.8 mm to (132.1, 81.6)
- moved C1 48.2 mm to (121.1, 92.0)
- moved C3 48.2 mm to (121.1, 90.2)
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Routing:
- net Data3: track 58.8 -> 116.4 mm
- net Data2: track 51.5 -> 105.6 mm
- net Data1: track 53.5 -> 89.0 mm
- net USART1_RX: track 40.8 -> 47.5 mm
- net VDD: track 204.5 -> 199.5 mm
- net +BATT: track 64.2 -> 69.2 mm
- net /VBAT_ADC: track 13.3 -> 16.5 mm
- net USART1_TX: track 43.9 -> 47.1 mm
- net Net-(U2-~{RST}): track 6.13 -> 5.16 mm
- net GND: vias 23 -> 24
Other:
- board outline removed
