File: Ksawer_Krzysztof.kicad_pcb (KiCad board)
At the start: 2 copper layers, 57 parts, among them J1 BAT, J3 V1, K1 1461103-1, K2 1461103-1, Q1 BC547, Q2 MMBT3904, Q3 MMBT3904, U1 DHT11, U2 ESP-12E, U3 NHD-C0220BIZ, U4 LTV-844, U5 STM32F038K6Ux, U6 TPS63021DSJR, U8 INA180A1, Y1 ABM3-B.000MHZ-D2Y

Commit message: gotowy_projekt
Parts:
- moved BZ1 0.13 mm to (112.8, 94.3)
Routing:
- net Data1: track 89.0 -> 93.8 mm
- net Data3: track 116.4 -> 120.2 mm
- net Data2: track 105.6 -> 108.8 mm
- net USART1_RX: track 47.5 -> 48.1 mm

Commit message: uj
Routing:
- net GND: track 57.2 -> 58.5 mm
- net /VBAT_ADC: track 16.5 -> 16.6 mm, vias 0 -> 2
Other:
- board outline added: 74.7 x 44.5 mm
Changed lines of the file:
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@@
     (property "TEXAS_INSTRUMENTS-PURCHASE-URL" "https://snapeda.com/shop?store=Texas+Instruments&id=296571")
     (attr smd)
-    (fp_text reference "U6" (at 0.0607 -3.03615) (layer "F.SilkS")
-        (effects (font (size 0.64 0.64) (thickness 0.15)))
+    (fp_text reference "U6" (at 0.0607 -3.54415) (layer "F.SilkS")
+        (effects (font (size 0.8 0.8) (thickness 0.15)))
     )
     (fp_text value "TPS63021DSJR" (at 4.096 3.1564) (layer "F.Fab")
@@
   )
   (gr_rect (start 88.646 77.216) (end 163.322 121.666)
-    (stroke (width 0.15) (type default)) (fill none) (layer "Dwgs.User"))
+    (stroke (width 0.1) (type default)) (fill none) (layer "Edge.Cuts"))
   (segment (start 123.9119 92.0319) (end 123.972 92.092) (width 0.4) (layer "F.Cu") (net 1))
   (segment (start 155.702 102.362) (end 154.432 101.092) (width 0.4) (layer "F.Cu") (net 1))
@@
   (segment (start 156.0576 118.27455) (end 156.90905 119.126) (width 0.4) (layer "F.Cu") (net 1))
   (segment (start 109.3724 89.271) (end 112.776 92.6746) (width 0.4) (layer "F.Cu") (net 1))
+  (segment (start 158.222 89.222) (end 157.222 89.222) (width 0.4) (layer "F.Cu") (net 1))
   (segment (start 162.56 92.456) (end 159.326 89.222) (width 0.4) (layer "F.Cu") (net 1))
+  (segment (start 143.6508 93.8392) (end 145.796 91.694) (width 0.4) (layer "F.Cu") (net 1))
   (segment (start 143.8656 99.7458) (end 144.0445 99.5669) (width 0.26) (layer "F.Cu") (net 1))
   (segment (start 95.965 89.662) (end 95.965 93.933) (width 0.4) (layer "F.Cu") (net 1))
@@
   (segment (start 98.6028 85.588) (end 98.6028 87.0104) (width 0.4) (layer "F.Cu") (net 1))
   (segment (start 138.9656 96.266) (end 140.6398 97.9402) (width 0.4) (layer "F.Cu") (net 1))
-  (segment (start 154.337 92.107) (end 153.924 91.694) (width 0.4) (layer "F.Cu") (net 1))
+  (segment (start 157.222 89.222) (end 154.845 91.599) (width 0.4) (layer "F.Cu") (net 1))
   (segment (start 157.226 102.362) (end 162.56 97.028) (width 0.4) (layer "F.Cu") (net 1))
   (segment (start 112.776 92.6746) (end 115.7886 89.662) (width 0.4) (layer "F.Cu") (net 1))
+  (segment (start 154.845 91.599) (end 152.972 93.472) (width 0.4) (layer "F.Cu") (net 1))
   (segment (start 119.333 80.4565) (end 119.333 85.899) (width 0.4) (layer "F.Cu") (net 1))
   (segment (start 119.333 85.899) (end 119.714 86.28) (width 0.4) (layer "F.Cu") (net 1))
-  (segment (start 143.6508 93.8392) (end 143.6508 99.1732) (width 0.4) (layer "F.Cu") (net 1))
   (segment (start 95.965 89.662) (end 95.965 88.2258) (width 0.4) (layer "F.Cu") (net 1))
   (segment (start 97.6299 84.6151) (end 97.6299 83.9801) (width 0.4) (layer "F.Cu") (net 1))
@@
   (segment (start 124.714 96.266) (end 138.9656 96.266) (width 0.4) (layer "F.Cu") (net 1))
   (segment (start 153.992 89.222) (end 150.7236 85.9536) (width 0.4) (layer "F.Cu") (net 1))
-  (segment (start 145.796 91.694) (end 143.6508 93.8392) (width 0.4) (layer "F.Cu") (net 1))
   (segment (start 119.968 86.534) (end 120.65 87.216) (width 0.4) (layer "F.Cu") (net 1))
   (segment (start 157.734 103.886) (end 157.226 103.378) (width 0.4) (layer "F.Cu") (net 1))
@@
   (segment (start 158.222 89.222) (end 153.992 89.222) (width 0.4) (layer "F.Cu") (net 1))
   (segment (start 98.6028 85.588) (end 97.6299 84.6151) (width 0.4) (layer "F.Cu") (net 1))
-  (segment (start 153.956 92.488) (end 152.972 93.472) (width 0.4) (layer "F.Cu") (net 1))
   (segment (start 121.92 91.9988) (end 124.3868 91.9988) (width 0.4) (layer "F.Cu") (net 1))
   (segment (start 121.92 93.472) (end 124.714 96.266) (width 0.4) (layer "F.Cu") (net 1))
@@
   (segment (start 150.7236 85.9536) (end 144.2701 85.9536) (width 0.4) (layer "F.Cu") (net 1))
   (segment (start 117.856 89.662) (end 119.714 87.804) (width 0.4) (layer "F.Cu") (net 1))
-  (segment (start 154.337 92.107) (end 153.956 92.488) (width 0.4) (layer "F.Cu") (net 1))
-  (segment (start 153.924 91.694) (end 145.796 91.694) (width 0.4) (layer "F.Cu") (net 1))
   (segment (start 140.9932 97.9402) (end 142.7988 99.7458) (width 0.26) (layer "F.Cu") (net 1))
   (segment (start 144.0445 99.5669) (end 145.896 101.4184) (width 0.26) (layer "F.Cu") (net 1))
@@
   (segment (start 115.7886 89.662) (end 117.856 89.662) (width 0.4) (layer "F.Cu") (net 1))
   (segment (start 157.734 108.712) (end 157.734 103.886) (width 0.4) (layer "F.Cu") (net 1))
+  (segment (start 154.75 91.694) (end 154.845 91.599) (width 0.4) (layer "F.Cu") (net 1))
   (segment (start 144.2701 85.9536) (end 144.2701 88.1361) (width 0.4) (layer "F.Cu") (net 1))
+  (segment (start 143.6508 99.1732) (end 143.6508 93.8392) (width 0.4) (layer "F.Cu") (net 1))
   (segment (start 103.886 89.271) (end 109.3724 89.271) (width 0.4) (layer "F.Cu") (net 1))
-  (segment (start 158.222 89.222) (end 157.222 89.222) (width 0.4) (layer "F.Cu") (net 1))
+  (segment (start 145.796 91.694) (end 154.75 91.694) (width 0.4) (layer "F.Cu") (net 1))
   (segment (start 157.226 103.378) (end 157.226 102.362) (width 0.4) (layer "F.Cu") (net 1))
   (segment (start 140.6398 97.9402) (end 140.9932 97.9402) (width 0.26) (layer "F.Cu") (net 1))
@@
   (segment (start 112.776 92.6746) (end 112.776 94.224) (width 0.4) (layer "F.Cu") (net 1))
   (segment (start 142.7988 99.7458) (end 143.8656 99.7458) (width 0.26) (layer "F.Cu") (net 1))
-  (segment (start 157.222 89.222) (end 154.337 92.107) (width 0.4) (layer "F.Cu") (net 1))
   (segment (start 95.965 93.933) (end 96.266 94.234) (width 0.4) (layer "F.Cu") (net 1))
   (segment (start 109.9566 81.4324) (end 109.9566 84.064) (width 0.26) (layer "F.Cu") (net 2))
@@
   (segment (start 147.066 112.66115) (end 147.162 112.56515) (width 0.4) (layer "F.Cu") (net 3))
   (segment (start 147.853 100.7309) (end 147.853 100.208304) (width 0.4) (layer "F.Cu") (net 3))
+  (segment (start 149.194 112.56515) (end 149.194 112.426) (width 0.4) (layer "F.Cu") (net 3))
   (segment (start 138.6586 110.9726) (end 138.684 110.998) (width 0.4) (layer "F.Cu") (net 3))
   (segment (start 140.5313 112.59185) (end 140.558 112.56515) (width 0.4) (layer "F.Cu") (net 3))
@@
   (segment (start 138.6586 109.8539) (end 138.6586 110.9726) (width 0.4) (layer "F.Cu") (net 3))
   (segment (start 138.7025 113.89885) (end 138.7025 112.64265) (width 0.4) (layer "F.Cu") (net 3))
-  (segment (start 148.522 89.222) (end 149.722 89.222) (width 0.4) (layer "F.Cu") (net 3))
   (segment (start 118.1872 101.3048) (end 119.5928 101.3048) (width 0.4) (layer "F.Cu") (net 3))
   (segment (start 142.2146 109.9058) (end 142.2146 110.9726) (width 0.4) (layer "F.Cu") (net 3))
@@
   (segment (start 132.96955 100.71155) (end 134.4941 99.187) (width 0.4) (layer "F.Cu") (net 3))
   (segment (start 142.1627 109.8539) (end 142.2146 109.9058) (width 0.4) (layer "F.Cu") (net 3))
+  (segment (start 149.194 112.426) (end 150.876 110.744) (width 0.4) (layer "F.Cu") (net 3))
   (segment (start 140.5313 113.89885) (end 140.5313 112.59185) (width 0.4) (layer "F.Cu") (net 3))
   (segment (start 149.0218 113.90795) (end 149.0218 112.73735) (width 0.4) (layer "F.Cu") (net 3))
@@
   (segment (start 121.158 80.4565) (end 121.158 78.232) (width 0.26) (layer "F.Cu") (net 4))
   (segment (start 150.368 95.504) (end 150.368 94.076) (width 0.26) (layer "F.Cu") (net 5))
-  (segment (start 150.368 94.076) (end 150.972 93.472) (width 0.2) (layer "F.Cu") (net 5))
+  (segment (start 150.368 94.076) (end 150.972 93.472) (width 0.26) (layer "F.Cu") (net 5))
   (segment (start 148.8043 93.6397) (end 148.972 93.472) (width 0.2) (layer "F.Cu") (net 6))
   (segment (start 148.844 93.6) (end 148.972 93.472) (width 0.2) (layer "F.Cu") (net 6))
@@
   (segment (start 140.3096 100.6432) (end 141.5848 101.9184) (width 0.26) (layer "F.Cu") (net 10))
   (segment (start 140.3096 104.3432) (end 140.3392 104.3432) (width 0.2) (layer "F.Cu") (net 11))
-  (segment (start 144.821 102.4184) (end 144.9324 102.4184) (width 0.2) (layer "F.Cu") (net 11))
   (segment (start 140.3392 104.3432) (end 142.2696 102.4128) (width 0.26) (layer "F.Cu") (net 11))
   (segment (start 136.2191 100.2527) (end 140.3096 104.3432) (width 0.26) (layer "F.Cu") (net 11))
@@
   (segment (start 155.798 114.08915) (end 157.195 114.08915) (width 0.26) (layer "F.Cu") (net 41))
   (segment (start 151.745 111.653) (end 153.11885 110.27915) (width 0.26) (layer "F.Cu") (net 42))
-  (segment (start 148.737 111.653) (end 151.745 111.653) (width 0.26) (layer "F.Cu") (net 42))
+  (segment (start 151.745 111.653) (end 151.638 111.76) (width 0.26) (layer "F.Cu") (net 42))
   (segment (start 145.542 108.458) (end 148.737 111.653) (width 0.26) (layer "F.Cu") (net 42))
   (segment (start 146.0684 103.9184) (end 145.542 104.4448) (width 0.26) (layer "F.Cu") (net 42))
@@
   (segment (start 146.6655 103.9184) (end 146.0684 103.9184) (width 0.26) (layer "F.Cu") (net 42))
   (segment (start 145.542 104.4448) (end 145.542 108.458) (width 0.26) (layer "F.Cu") (net 42))
+  (via (at 148.737 111.653) (size 0.75) (drill 0.5) (layers "F.Cu" "B.Cu") (net 42))
+  (via (at 151.638 111.76) (size 0.75) (drill 0.5) (layers "F.Cu" "B.Cu") (net 42))
+  (segment (start 148.844 111.76) (end 148.737 111.653) (width 0.26) (layer "B.Cu") (net 42))
+  (segment (start 151.638 111.76) (end 148.844 111.76) (width 0.26) (layer "B.Cu") (net 42))
   (segment (start 140.43 80.092) (end 139.68 80.092) (width 0.2) (layer "F.Cu") (net 57))
   (segment (start 142.24 81.902) (end 140.43 80.092) (width 0.26) (layer "F.Cu") (net 57))
